Commit message: added fingertip positions to urdf, support for ros1 and ros2

File: models/urdf/orcahand_left.urdf (robot description, URDF)
Before this commit: robot orcahand_left, 37 links, 36 joints
Links:
- added link left_index_fingertip, mass 0.0
- added link left_middle_fingertip, mass 0.0
- added link left_pinky_fingertip, mass 0.0
- added link left_ring_fingertip, mass 0.0
- added link left_thumb_fingertip, mass 0.0
Joints:
- added joint left_index_ip2left_index_fingertip_fixed_offset: type fixed, parent left_index_ip, child left_index_fingertip, origin xyz=0.009 0.0 0.035 rpy=0.0 0.0 0.0
- added joint left_middle_ip2left_index_fingertip_fixed_offset: type fixed, parent left_middle_ip, child left_middle_fingertip, origin xyz=0.009 0.0 0.035 rpy=0.0 0.0 0.0
- added joint left_pinky_ip2left_index_fingertip_fixed_offset: type fixed, parent left_pinky_ip, child left_pinky_fingertip, origin xyz=0.009 0.0 0.035 rpy=0.0 0.0 0.0
- added joint left_ring_ip2left_index_fingertip_fixed_offset: type fixed, parent left_ring_ip, child left_ring_fingertip, origin xyz=0.009 0.0 0.035 rpy=0.0 0.0 0.0
- added joint thumb_dp2left_thumb_fingertip_fixed_offset: type fixed, parent left_thumb_dp, child left_thumb_fingertip, origin xyz=0.003 0.0 0.025 rpy=0.0 0.0 0.0

File: models/urdf/orcahand_left_extended.urdf (robot description, URDF)
Before this commit: robot orcahand_left_extended, 37 links, 36 joints
Links:
- added link left_index_fingertip, mass 0.0
- added link left_middle_fingertip, mass 0.0
- added link left_pinky_fingertip, mass 0.0
- added link left_ring_fingertip, mass 0.0
- added link left_thumb_fingertip, mass 0.0
Joints:
- added joint left_index_ip2left_index_fingertip_fixed_offset: type fixed, parent left_index_ip, child left_index_fingertip, origin xyz=0.009 0.0 0.035 rpy=0.0 0.0 0.0
- added joint left_middle_ip2left_index_fingertip_fixed_offset: type fixed, parent left_middle_ip, child left_middle_fingertip, origin xyz=0.009 0.0 0.035 rpy=0.0 0.0 0.0
- added joint left_pinky_ip2left_index_fingertip_fixed_offset: type fixed, parent left_pinky_ip, child left_pinky_fingertip, origin xyz=0.009 0.0 0.035 rpy=0.0 0.0 0.0
- added joint left_ring_ip2left_index_fingertip_fixed_offset: type fixed, parent left_ring_ip, child left_ring_fingertip, origin xyz=0.009 0.0 0.035 rpy=0.0 0.0 0.0
- added joint thumb_dp2left_thumb_fingertip_fixed_offset: type fixed, parent left_thumb_dp, child left_thumb_fingertip, origin xyz=0.003 0.0 0.025 rpy=0.0 0.0 0.0

File: models/urdf/orcahand_right.urdf (robot description, URDF)
Before this commit: robot orcahand_right_extended, 37 links, 36 joints
Links:
- added link right_index_fingertip, mass 0.0
- added link right_middle_fingertip, mass 0.0
- added link right_pinky_fingertip, mass 0.0
- added link right_ring_fingertip, mass 0.0
- added link right_thumb_fingertip, mass 0.0
Joints:
- added joint right_index_ip2right_index_fingertip_fixed_offset: type fixed, parent right_index_ip, child right_index_fingertip, origin xyz=-0.009 0.0 0.035 rpy=0.0 0.0 0.0
- added joint right_middle_ip2right_index_fingertip_fixed_offset: type fixed, parent right_middle_ip, child right_middle_fingertip, origin xyz=-0.009 0.0 0.035 rpy=0.0 0.0 0.0
- added joint right_pinky_ip2right_index_fingertip_fixed_offset: type fixed, parent right_pinky_ip, child right_pinky_fingertip, origin xyz=-0.009 0.0 0.035 rpy=0.0 0.0 0.0
- added joint right_ring_ip2right_index_fingertip_fixed_offset: type fixed, parent right_ring_ip, child right_ring_fingertip, origin xyz=-0.009 0.0 0.035 rpy=0.0 0.0 0.0
- added joint thumb_dp2right_thumb_fingertip_fixed_offset: type fixed, parent right_thumb_dp, child right_thumb_fingertip, origin xyz=-0.003 0.0 0.025 rpy=0.0 0.0 0.0

File: models/urdf/orcahand_right_extended.urdf (robot description, URDF)
Before this commit: robot orcahand_right_extended, 37 links, 36 joints
Links:
- added link right_index_fingertip, mass 0.0
- added link right_middle_fingertip, mass 0.0
- added link right_pinky_fingertip, mass 0.0
- added link right_ring_fingertip, mass 0.0
- added link right_thumb_fingertip, mass 0.0
Joints:
- added joint right_index_ip2right_index_fingertip_fixed_offset: type fixed, parent right_index_ip, child right_index_fingertip, origin xyz=-0.009 0.0 0.035 rpy=0.0 0.0 0.0
- added joint right_middle_ip2right_index_fingertip_fixed_offset: type fixed, parent right_middle_ip, child right_middle_fingertip, origin xyz=-0.009 0.0 0.035 rpy=0.0 0.0 0.0
- added joint right_pinky_ip2right_index_fingertip_fixed_offset: type fixed, parent right_pinky_ip, child right_pinky_fingertip, origin xyz=-0.009 0.0 0.035 rpy=0.0 0.0 0.0
- added joint right_ring_ip2right_index_fingertip_fixed_offset: type fixed, parent right_ring_ip, child right_ring_fingertip, origin xyz=-0.009 0.0 0.035 rpy=0.0 0.0 0.0
- added joint thumb_dp2right_thumb_fingertip_fixed_offset: type fixed, parent right_thumb_dp, child right_thumb_fingertip, origin xyz=-0.003 0.0 0.025 rpy=0.0 0.0 0.0

Commit message: joint limit and zero position fixes for v1

File: models/urdf/orcahand_left.urdf (robot description, URDF)
Before this commit: robot orcahand_left, 42 links, 41 joints
Joints:
- joint left_index_abd: limit lower=-1.04577 upper=0.24577 effort=100 velocity=100 -> lower=-0.645772 upper=0.645772 effort=100 velocity=100
- joint left_index_mcp: limit lower=-0.34907 upper=1.65806 effort=100 velocity=100 -> lower=-0.349066 upper=1.658063 effort=100 velocity=100
- joint left_index_pip: limit lower=-0.34907 upper=1.88496 effort=100 velocity=100 -> lower=-0.349066 upper=1.884956 effort=100 velocity=100
- joint left_middle_abd: limit lower=-0.64577 upper=0.64577 effort=100 velocity=100 -> lower=-0.645772 upper=0.645772 effort=100 velocity=100
- joint left_middle_mcp: limit lower=-0.34907 upper=1.58825 effort=100 velocity=100 -> lower=-0.349066 upper=1.588250 effort=100 velocity=100
- joint left_middle_pip: limit lower=-0.34907 upper=1.8675 effort=100 velocity=100 -> lower=-0.349066 upper=1.884956 effort=100 velocity=100
- joint left_pinky_abd: limit lower=-0.12244 upper=1.1691 effort=100 velocity=100 -> lower=-0.645772 upper=0.645772 effort=100 velocity=100
- joint left_pinky_mcp: limit lower=-0.34907 upper=1.71042 effort=100 velocity=100 -> lower=-0.349066 upper=1.727876 effort=100 velocity=100
- joint left_pinky_pip: limit lower=-0.34907 upper=1.88496 effort=100 velocity=100 -> lower=-0.349066 upper=1.884956 effort=100 velocity=100
- joint left_ring_abd: limit lower=-0.47577 upper=0.80577 effort=100 velocity=100 -> lower=-0.541052 upper=0.645772 effort=100 velocity=100
- joint left_ring_mcp: limit lower=-0.34907 upper=1.58825 effort=100 velocity=100 -> lower=-0.349066 upper=1.588250 effort=100 velocity=100
- joint left_ring_pip: limit lower=-0.34907 upper=1.8675 effort=100 velocity=100 -> lower=-0.349066 upper=1.884956 effort=100 velocity=100
- joint left_thumb_abd: limit lower=-1.08211 upper=0.0 effort=100 velocity=100 -> lower=-0.349066 upper=0.733038 effort=100 velocity=100
- joint left_thumb_dip: limit lower=-0.85384 upper=1.45 effort=100 velocity=100 -> lower=-0.349066 upper=1.954769 effort=100 velocity=100
- joint left_thumb_mcp: limit lower=-0.87266 upper=0.87266 effort=100 velocity=100 -> lower=-0.610865 upper=1.134464 effort=100 velocity=100
- joint left_thumb_pip: limit lower=-0.7944 upper=1.23 effort=100 velocity=100 -> lower=-0.209440 upper=1.884956 effort=100 velocity=100
- joint left_wrist: limit lower=-0.8972 upper=0.6736 effort=100 velocity=100 -> lower=-1.047198 upper=0.523599 effort=100 velocity=100

File: models/urdf/orcahand_left_extended.urdf (robot description, URDF)
Before this commit: robot orcahand_left_extended, 42 links, 41 joints
Joints:
- joint left_index_abd: limit lower=-1.04577 upper=0.24577 effort=100 velocity=100 -> lower=-0.645772 upper=0.645772 effort=100 velocity=100
- joint left_index_mcp: limit lower=-0.34907 upper=1.65806 effort=100 velocity=100 -> lower=-0.349066 upper=1.658063 effort=100 velocity=100
- joint left_index_pip: limit lower=-0.34907 upper=1.88496 effort=100 velocity=100 -> lower=-0.349066 upper=1.884956 effort=100 velocity=100
- joint left_middle_abd: limit lower=-0.64577 upper=0.64577 effort=100 velocity=100 -> lower=-0.645772 upper=0.645772 effort=100 velocity=100
- joint left_middle_mcp: limit lower=-0.34907 upper=1.58825 effort=100 velocity=100 -> lower=-0.349066 upper=1.588250 effort=100 velocity=100
- joint left_middle_pip: limit lower=-0.34907 upper=1.8675 effort=100 velocity=100 -> lower=-0.349066 upper=1.884956 effort=100 velocity=100
- joint left_pinky_abd: limit lower=-0.12244 upper=1.1691 effort=100 velocity=100 -> lower=-0.645772 upper=0.645772 effort=100 velocity=100
- joint left_pinky_mcp: limit lower=-0.34907 upper=1.71042 effort=100 velocity=100 -> lower=-0.349066 upper=1.727876 effort=100 velocity=100
- joint left_pinky_pip: limit lower=-0.34907 upper=1.88496 effort=100 velocity=100 -> lower=-0.349066 upper=1.884956 effort=100 velocity=100
- joint left_ring_abd: limit lower=-0.47577 upper=0.80577 effort=100 velocity=100 -> lower=-0.541052 upper=0.645772 effort=100 velocity=100
- joint left_ring_mcp: limit lower=-0.34907 upper=1.58825 effort=100 velocity=100 -> lower=-0.349066 upper=1.588250 effort=100 velocity=100
- joint left_ring_pip: limit lower=-0.34907 upper=1.8675 effort=100 velocity=100 -> lower=-0.349066 upper=1.884956 effort=100 velocity=100
- joint left_thumb_abd: limit lower=-1.08211 upper=0.0 effort=100 velocity=100 -> lower=-0.349066 upper=0.733038 effort=100 velocity=100
- joint left_thumb_dip: limit lower=-0.85384 upper=1.45 effort=100 velocity=100 -> lower=-0.349066 upper=1.954769 effort=100 velocity=100
- joint left_thumb_mcp: limit lower=-0.87266 upper=0.87266 effort=100 velocity=100 -> lower=-0.610865 upper=1.134464 effort=100 velocity=100
- joint left_thumb_pip: limit lower=-0.7944 upper=1.23 effort=100 velocity=100 -> lower=-0.209440 upper=1.884956 effort=100 velocity=100
- joint left_wrist: limit lower=-0.8972 upper=0.6736 effort=100 velocity=100 -> lower=-1.047198 upper=0.523599 effort=100 velocity=100

File: models/urdf/orcahand_right.urdf (robot description, URDF)
Before this commit: robot orcahand_right, 42 links, 41 joints
Joints:
- joint right_index_abd: limit lower=-1.04577 upper=0.24577 effort=100 velocity=100 -> lower=-0.645772 upper=0.645772 effort=100 velocity=100
- joint right_index_mcp: limit lower=-0.34907 upper=1.65806 effort=100 velocity=100 -> lower=-0.349066 upper=1.658063 effort=100 velocity=100
- joint right_index_pip: limit lower=-0.34907 upper=1.88496 effort=100 velocity=100 -> lower=-0.349066 upper=1.884956 effort=100 velocity=100
- joint right_middle_abd: limit lower=-0.64577 upper=0.64577 effort=100 velocity=100 -> lower=-0.645772 upper=0.645772 effort=100 velocity=100
- joint right_middle_mcp: limit lower=-0.34907 upper=1.58825 effort=100 velocity=100 -> lower=-0.349066 upper=1.588250 effort=100 velocity=100
- joint right_middle_pip: limit lower=-0.34907 upper=1.8675 effort=100 velocity=100 -> lower=-0.349066 upper=1.884956 effort=100 velocity=100
- joint right_pinky_abd: limit lower=-0.12244 upper=1.1691 effort=100 velocity=100 -> lower=-0.645772 upper=0.645772 effort=100 velocity=100
- joint right_pinky_mcp: limit lower=-0.34907 upper=1.71042 effort=100 velocity=100 -> lower=-0.349066 upper=1.727876 effort=100 velocity=100
- joint right_pinky_pip: limit lower=-0.34907 upper=1.88496 effort=100 velocity=100 -> lower=-0.349066 upper=1.884956 effort=100 velocity=100
- joint right_ring_abd: limit lower=-0.47577 upper=0.80577 effort=100 velocity=100 -> lower=-0.541052 upper=0.645772 effort=100 velocity=100
- joint right_ring_mcp: limit lower=-0.34907 upper=1.58825 effort=100 velocity=100 -> lower=-0.349066 upper=1.588250 effort=100 velocity=100
- joint right_ring_pip: limit lower=-0.34907 upper=1.8675 effort=100 velocity=100 -> lower=-0.349066 upper=1.884956 effort=100 velocity=100
- joint right_thumb_abd: limit lower=-1.08211 upper=0.0 effort=100 velocity=100 -> lower=-0.349066 upper=0.733038 effort=100 velocity=100
- joint right_thumb_dip: limit lower=-0.85384 upper=1.45 effort=100 velocity=100 -> lower=-0.349066 upper=1.954769 effort=100 velocity=100
- joint right_thumb_mcp: limit lower=-0.87266 upper=0.87266 effort=100 velocity=100 -> lower=-0.610865 upper=1.134464 effort=100 velocity=100
- joint right_thumb_pip: limit lower=-0.7944 upper=1.23 effort=100 velocity=100 -> lower=-0.209440 upper=1.884956 effort=100 velocity=100
- joint right_wrist: axis 1.0 0.0 0.0 -> -1.0 0.0 0.0; limit lower=-0.6736 upper=0.8972 effort=100 velocity=100 -> lower=-1.047198 upper=0.523599 effort=100 velocity=100

File: models/urdf/orcahand_right_extended.urdf (robot description, URDF)
Before this commit: robot orcahand_right_extended, 42 links, 41 joints
Joints:
- joint right_index_abd: limit lower=-1.04577 upper=0.24577 effort=100 velocity=100 -> lower=-0.645772 upper=0.645772 effort=100 velocity=100
- joint right_index_mcp: limit lower=-0.34907 upper=1.65806 effort=100 velocity=100 -> lower=-0.349066 upper=1.658063 effort=100 velocity=100
- joint right_index_pip: limit lower=-0.34907 upper=1.88496 effort=100 velocity=100 -> lower=-0.349066 upper=1.884956 effort=100 velocity=100
- joint right_middle_abd: limit lower=-0.64577 upper=0.64577 effort=100 velocity=100 -> lower=-0.645772 upper=0.645772 effort=100 velocity=100
- joint right_middle_mcp: limit lower=-0.34907 upper=1.58825 effort=100 velocity=100 -> lower=-0.349066 upper=1.588250 effort=100 velocity=100
- joint right_middle_pip: limit lower=-0.34907 upper=1.8675 effort=100 velocity=100 -> lower=-0.349066 upper=1.884956 effort=100 velocity=100
- joint right_pinky_abd: limit lower=-0.12244 upper=1.1691 effort=100 velocity=100 -> lower=-0.645772 upper=0.645772 effort=100 velocity=100
- joint right_pinky_mcp: limit lower=-0.34907 upper=1.71042 effort=100 velocity=100 -> lower=-0.349066 upper=1.727876 effort=100 velocity=100
- joint right_pinky_pip: limit lower=-0.34907 upper=1.88496 effort=100 velocity=100 -> lower=-0.349066 upper=1.884956 effort=100 velocity=100
- joint right_ring_abd: limit lower=-0.47577 upper=0.80577 effort=100 velocity=100 -> lower=-0.541052 upper=0.645772 effort=100 velocity=100
- joint right_ring_mcp: limit lower=-0.34907 upper=1.58825 effort=100 velocity=100 -> lower=-0.349066 upper=1.588250 effort=100 velocity=100
- joint right_ring_pip: limit lower=-0.34907 upper=1.8675 effort=100 velocity=100 -> lower=-0.349066 upper=1.884956 effort=100 velocity=100
- joint right_thumb_abd: limit lower=-1.08211 upper=0.0 effort=100 velocity=100 -> lower=-0.349066 upper=0.733038 effort=100 velocity=100
- joint right_thumb_dip: limit lower=-0.85384 upper=1.45 effort=100 velocity=100 -> lower=-0.349066 upper=1.954769 effort=100 velocity=100
- joint right_thumb_mcp: limit lower=-0.87266 upper=0.87266 effort=100 velocity=100 -> lower=-0.610865 upper=1.134464 effort=100 velocity=100
- joint right_thumb_pip: limit lower=-0.7944 upper=1.23 effort=100 velocity=100 -> lower=-0.209440 upper=1.884956 effort=100 velocity=100
- joint right_wrist: axis 1.0 0.0 0.0 -> -1.0 0.0 0.0; limit lower=-0.6736 upper=0.8972 effort=100 velocity=100 -> lower=-1.047198 upper=0.523599 effort=100 velocity=100
