Commit message: Remove spurious -35 deg roll from the right wrist URDF origin
The URDF carried rpy=(-0.6109, 0, -pi/2) on the wrist joint origin while the
MJCF never had it (b7fbfce zeroed the wrist ref). The roll is mathematically
identical to pinning the wrist at its +35 deg travel limit (0.0000 mm
difference) and made URDF zero-pose disagree with MuJoCo and with
orca_core's extracted kinematics. Both URDFs and both MJCFs are now
roll-free at the wrist.

Co-Authored-By: Claude Fable 5 <noreply@anthropic.com>

File: v2/models/urdf/orcahand_right.urdf (robot description, URDF)
Before this commit: robot orcahand_right, 19 links, 18 joints
Joints:
- joint R-Carpals_8d1f1041_to_TopTower-Model_4a80d30e: origin xyz=5.551115123125783e-17 2.3418766925686896e-17 0.04000000000000006 rpy=-0.610865285723758 0.0 -1.5707963267948992 -> xyz=5.551115123125783e-17 2.3418766925686896e-17 0.04000000000000006 rpy=0.0 0.0 -1.5707963267948992
